Commit message: Body.urdf is updated and genarate.py now geneartes a robot with two legs and a torso.

File: body.urdf (robot description, URDF)
Before this commit: robot robot, 2 links, 0 joints
Links:
- removed link Leg
- added link BackLeg, mass 1; collision box size=1 1 1; visual box size=1 1 1
- added link FrontLeg, mass 1; collision box size=1 1 1; visual box size=1 1 1
Joints:
- added joint Torso_BackLeg: type revolute, parent Torso, child BackLeg, origin xyz=1.0 0 1.0 rpy=0 0 0, axis 0 1 0, limit lower=-3.14159 upper=3.14159 effort=0.0 velocity=0.0
- added joint Torso_FrontLeg: type revolute, parent Torso, child FrontLeg, origin xyz=2.0 0 1.0 rpy=0 0 0, axis 0 1 0, limit lower=-3.14159 upper=3.14159 effort=0.0 velocity=0.0

Commit message: Quad formed

File: body.urdf (robot description, URDF)
Before this commit: robot robot, 3 links, 2 joints
Links:
- added link BackLowerLeg, mass 1; collision box size=0.2 0.2 1; visual box size=0.2 0.2 1
- added link FrontLowerLeg, mass 1; collision box size=0.2 0.2 1; visual box size=0.2 0.2 1
- added link LeftLeg, mass 1; collision box size=1 0.2 0.2; visual box size=1 0.2 0.2
- added link LeftLowerLeg, mass 1; collision box size=0.2 0.2 1; visual box size=0.2 0.2 1
- added link RightLeg, mass 1; collision box size=1 0.2 0.2; visual box size=1 0.2 0.2
- added link RightLowerLeg, mass 1; collision box size=0.2 0.2 1; visual box size=0.2 0.2 1
- link BackLeg: geometry collision box size=0.2 1 0.2; visual box size=0.2 1 0.2
- link FrontLeg: geometry collision box size=0.2 1 0.2; visual box size=0.2 1 0.2
Joints:
- added joint BackLeg_BackLowerLeg: type revolute, parent BackLeg, child BackLowerLeg, origin xyz=0 -1 0 rpy=0 0 0, axis 0 1 0, limit lower=-3.14159 upper=3.14159 effort=0.0 velocity=0.0
- added joint FrontLeg_FrontLowerLeg: type revolute, parent FrontLeg, child FrontLowerLeg, origin xyz=0 1 0 rpy=0 0 0, axis 0 1 0, limit lower=-3.14159 upper=3.14159 effort=0.0 velocity=0.0
- added joint LeftLeg_LeftLowerLeg: type revolute, parent LeftLeg, child LeftLowerLeg, origin xyz=-1 0 0 rpy=0 0 0, axis 0 1 0, limit lower=-3.14159 upper=3.14159 effort=0.0 velocity=0.0
- added joint RightLeg_RightLowerLeg: type revolute, parent RightLeg, child RightLowerLeg, origin xyz=1 0 0 rpy=0 0 0, axis 0 1 0, limit lower=-3.14159 upper=3.14159 effort=0.0 velocity=0.0
- added joint Torso_LeftLeg: type revolute, parent Torso, child LeftLeg, origin xyz=-0.5 0 1.0 rpy=0 0 0, axis 0 1 0, limit lower=-3.14159 upper=3.14159 effort=0.0 velocity=0.0
- added joint Torso_RightLeg: type revolute, parent Torso, child RightLeg, origin xyz=0.5 0 1.0 rpy=0 0 0, axis 0 1 0, limit lower=-3.14159 upper=3.14159 effort=0.0 velocity=0.0
- joint Torso_BackLeg: axis 0 1 0 -> 1 0 0; origin xyz=1.0 0 1.0 rpy=0 0 0 -> xyz=0 -0.5 1.0 rpy=0 0 0
- joint Torso_FrontLeg: axis 0 1 0 -> 1 0 0; origin xyz=2.0 0 1.0 rpy=0 0 0 -> xyz=0 0.5 1.0 rpy=0 0 0

Commit message: Vibing in the quad

File: body.urdf (robot description, URDF)
Before this commit: robot robot, 9 links, 8 joints
Joints:
- joint Torso_BackLeg: axis 1 0 0 -> 0 1 0
- joint Torso_FrontLeg: axis 1 0 0 -> 0 1 0

Commit message: Final projectgit add .

File: body.urdf (robot description, URDF)
Before this commit: robot robot, 9 links, 8 joints
Joints:
- joint BackLeg_BackLowerLeg: axis 0 1 0 -> 1 0 0
- joint FrontLeg_FrontLowerLeg: axis 0 1 0 -> 1 0 0
- joint Torso_BackLeg: axis 0 1 0 -> 1 0 0
- joint Torso_FrontLeg: axis 0 1 0 -> 1 0 0

Commit message: Much nicer looking dog

File: body.urdf (robot description, URDF)
Before this commit: robot robot, 9 links, 8 joints
Links:
- removed link BackLeg
- removed link BackLowerLeg
- removed link FrontLeg
- removed link FrontLowerLeg
- removed link LeftLeg
- removed link LeftLowerLeg
- removed link RightLeg
- removed link RightLowerLeg
- added link BackLeftLowerArm, mass 1; collision box size=1 0.25 0.25; visual box size=1 0.25 0.25
- added link BackLeftShoulder, mass 1; collision box size=0.5 0.5 0.5; visual box size=0.5 0.5 0.5
- added link BackLeftUpperArm, mass 1; collision box size=1 0.25 0.25; visual box size=1 0.25 0.25
- added link BackRightLowerArm, mass 1; collision box size=1 0.25 0.25; visual box size=1 0.25 0.25
- added link BackRightShoulder, mass 1; collision box size=0.5 0.5 0.5; visual box size=0.5 0.5 0.5
- added link BackRightUpperArm, mass 1; collision box size=1 0.25 0.25; visual box size=1 0.25 0.25
- added link FrontLeftLowerArm, mass 1; collision box size=1 0.25 0.25; visual box size=1 0.25 0.25
- added link FrontLeftShoulder, mass 1; collision box size=0.5 0.5 0.5; visual box size=0.5 0.5 0.5
- added link FrontLeftUpperArm, mass 1; collision box size=1 0.25 0.25; visual box size=1 0.25 0.25
- added link FrontRightLowerArm, mass 1; collision box size=1 0.25 0.25; visual box size=1 0.25 0.25
- added link FrontRightShoulder, mass 1; collision box size=0.5 0.5 0.5; visual box size=0.5 0.5 0.5
- added link FrontRightUpperArm, mass 1; collision box size=1 0.25 0.25; visual box size=1 0.25 0.25
- link Torso: geometry collision box size=2 1 0.5; visual box size=2 1 0.5
Joints:
- removed joint BackLeg_BackLowerLeg
- removed joint FrontLeg_FrontLowerLeg
- removed joint LeftLeg_LeftLowerLeg
- removed joint RightLeg_RightLowerLeg
- removed joint Torso_BackLeg
- removed joint Torso_FrontLeg
- removed joint Torso_LeftLeg
- removed joint Torso_RightLeg
- added joint BackLeftShoulder_BackLeftUpperArm: type revolute, parent BackLeftShoulder, child BackLeftUpperArm, origin xyz=0 0 0 rpy=0 0 0, axis 0 1 0, limit lower=-3.14159 upper=3.14159 effort=0.0 velocity=0.0
- added joint BackLeftUpperArm_BackLeftLowerArm: type revolute, parent BackLeftUpperArm, child BackLeftLowerArm, origin xyz=-1 0 0 rpy=0 0 0, axis 0 1 0, limit lower=-3.14159 upper=3.14159 effort=0.0 velocity=0.0
- added joint BackRightShoulder_BackRightUpperArm: type revolute, parent BackRightShoulder, child BackRightUpperArm, origin xyz=0 0 0 rpy=0 0 0, axis 0 1 0, limit lower=-3.14159 upper=3.14159 effort=0.0 velocity=0.0
- added joint BackRightUpperArm_BackRightLowerArm: type revolute, parent BackRightUpperArm, child BackRightLowerArm, origin xyz=-1 0 0 rpy=0 0 0, axis 0 1 0, limit lower=-3.14159 upper=3.14159 effort=0.0 velocity=0.0
- added joint FrontLeftShoulder_FrontLeftUpperArm: type revolute, parent FrontLeftShoulder, child FrontLeftUpperArm, origin xyz=0 0 0 rpy=0 0 0, axis 0 1 0, limit lower=-3.14159 upper=3.14159 effort=0.0 velocity=0.0
- added joint FrontLeftUpperArm_FrontLeftLowerArm: type revolute, parent FrontLeftUpperArm, child FrontLeftLowerArm, origin xyz=-1 0 0 rpy=0 0 0, axis 0 1 0, limit lower=-3.14159 upper=3.14159 effort=0.0 velocity=0.0
- added joint FrontRightShoulder_FrontRightUpperArm: type revolute, parent FrontRightShoulder, child FrontRightUpperArm, origin xyz=0 0 0 rpy=0 0 0, axis 0 1 0, limit lower=-3.14159 upper=3.14159 effort=0.0 velocity=0.0
- added joint FrontRightUpperArm_FrontRightLowerArm: type revolute, parent FrontRightUpperArm, child FrontRightLowerArm, origin xyz=-1 0 0 rpy=0 0 0, axis 0 1 0, limit lower=-3.14159 upper=3.14159 effort=0.0 velocity=0.0
- added joint Torso_BackLeftShoulder: type revolute, parent Torso, child BackLeftShoulder, origin xyz=-0.75 0.5 1.0 rpy=0 0 0, axis 1 0 0, limit lower=-3.14159 upper=3.14159 effort=0.0 velocity=0.0
- added joint Torso_BackRightShoulder: type revolute, parent Torso, child BackRightShoulder, origin xyz=-0.75 -0.5 1.0 rpy=0 0 0, axis 1 0 0, limit lower=-3.14159 upper=3.14159 effort=0.0 velocity=0.0
- added joint Torso_FrontLeftShoulder: type revolute, parent Torso, child FrontLeftShoulder, origin xyz=0.75 0.5 1.0 rpy=0 0 0, axis 1 0 0, limit lower=-3.14159 upper=3.14159 effort=0.0 velocity=0.0
- added joint Torso_FrontRightShoulder: type revolute, parent Torso, child FrontRightShoulder, origin xyz=0.75 -0.5 1.0 rpy=0 0 0, axis 1 0 0, limit lower=-3.14159 upper=3.14159 effort=0.0 velocity=0.0

Commit message: Add weights file to store best of last run

File: body.urdf (robot description, URDF)
Before this commit: robot robot, 13 links, 12 joints
Links:
- added link Head, mass 1; collision box size=0.5 0.75 0.5; visual box size=0.5 0.75 0.5
- link BackLeftLowerArm: geometry collision box size=0.25 0.25 1; visual box size=0.25 0.25 1
- link BackRightLowerArm: geometry collision box size=0.25 0.25 1; visual box size=0.25 0.25 1
- link FrontLeftLowerArm: geometry collision box size=0.25 0.25 1; visual box size=0.25 0.25 1
- link FrontRightLowerArm: geometry collision box size=0.25 0.25 1; visual box size=0.25 0.25 1
Joints:
- added joint Torso_Head: type revolute, parent Torso, child Head, origin xyz=1 0 0.5 rpy=0 0 0, axis 1 0 0, limit lower=-3.14159 upper=3.14159 effort=0.0 velocity=0.0

Commit message: 3-d circles are being generated, SPHERES

File: body.urdf (robot description, URDF)
Before this commit: robot robot, 14 links, 13 joints
Links:
- link BackLeftLowerArm: mass 1 -> 1.0
- link BackLeftShoulder: mass 1 -> 1.0
- link BackLeftUpperArm: mass 1 -> 1.0
- link BackRightLowerArm: mass 1 -> 1.0
- link BackRightShoulder: mass 1 -> 1.0
- link BackRightUpperArm: mass 1 -> 1.0
- link FrontLeftLowerArm: mass 1 -> 1.0
- link FrontLeftShoulder: mass 1 -> 1.0
- link FrontLeftUpperArm: mass 1 -> 1.0
- link FrontRightLowerArm: mass 1 -> 1.0
- link FrontRightShoulder: mass 1 -> 1.0
- link FrontRightUpperArm: mass 1 -> 1.0
- link Head: mass 1 -> 1.0; geometry collision sphere radius=0.5; visual sphere radius=0.5
- link Torso: mass 1 -> 1.0

Commit message: Fitness calculation changed, playing with how to get the dog to stay level while walking

File: body.urdf (robot description, URDF)
Before this commit: robot robot, 14 links, 13 joints
Links:
- added link BackLeftKnee, mass 1.0; collision sphere radius=0.2; visual sphere radius=0.2
- added link BackRightKnee, mass 1.0; collision sphere radius=0.2; visual sphere radius=0.2
- added link FrontLeftKnee, mass 1.0; collision sphere radius=0.2; visual sphere radius=0.2
- added link FrontRightKnee, mass 1.0; collision sphere radius=0.2; visual sphere radius=0.2
- link BackLeftLowerArm: mass 1.0 -> 6
- link BackLeftShoulder: mass 1.0 -> 3
- link BackLeftUpperArm: mass 1.0 -> 2
- link BackRightLowerArm: mass 1.0 -> 6
- link BackRightShoulder: mass 1.0 -> 3
- link BackRightUpperArm: mass 1.0 -> 2
- link FrontLeftLowerArm: mass 1.0 -> 4
- link FrontLeftShoulder: mass 1.0 -> 3
- link FrontLeftUpperArm: mass 1.0 -> 2
- link FrontRightLowerArm: mass 1.0 -> 4
- link FrontRightShoulder: mass 1.0 -> 3
- link FrontRightUpperArm: mass 1.0 -> 2
- link Head: mass 1.0 -> 1
- link Torso: mass 1.0 -> 10
Joints:
- added joint BackLeftUpperArm_BackLeftKnee: type revolute, parent BackLeftUpperArm, child BackLeftKnee, origin xyz=0 0 0 rpy=0 0 0, axis 0 1 0, limit lower=-3.14159 upper=3.14159 effort=0.0 velocity=0.0
- added joint BackRightUpperArm_FrontRightKnee: type revolute, parent BackRightUpperArm, child BackRightKnee, origin xyz=0 0 0 rpy=0 0 0, axis 0 1 0, limit lower=-3.14159 upper=3.14159 effort=0.0 velocity=0.0
- added joint FrontLeftUpperArm_FrontLeftKnee: type revolute, parent FrontLeftUpperArm, child FrontLeftKnee, origin xyz=0 0 0 rpy=0 0 0, axis 0 1 0, limit lower=-3.14159 upper=3.14159 effort=0.0 velocity=0.0
- added joint FrontRightUpperArm_FrontRightKnee: type revolute, parent FrontRightUpperArm, child FrontRightKnee, origin xyz=0 0 0 rpy=0 0 0, axis 0 1 0, limit lower=-3.14159 upper=3.14159 effort=0.0 velocity=0.0

Commit message: Test

File: body.urdf (robot description, URDF)
Before this commit: robot robot, 18 links, 17 joints
Links:
- link BackLeftLowerArm: mass 6 -> 2
- link BackLeftShoulder: mass 3 -> 1
- link BackLeftUpperArm: mass 2 -> 1
- link BackRightLowerArm: mass 6 -> 2
- link BackRightShoulder: mass 3 -> 1
- link BackRightUpperArm: mass 2 -> 1
- link FrontLeftLowerArm: mass 4 -> 2
- link FrontLeftShoulder: mass 3 -> 1
- link FrontLeftUpperArm: mass 2 -> 1
- link FrontRightLowerArm: mass 4 -> 2
- link FrontRightShoulder: mass 3 -> 1
- link FrontRightUpperArm: mass 2 -> 1
- link Torso: mass 10 -> 1
